File: KiCad/ProjetCpatKiCad/ProjetCpatKiCad/ProjetCpatKiCad.kicad_sch (KiCad schematic)
At the start: 4 parts, among them J1 Power, J2 Digital/PWM, J3 Analog, J4 Digital/PWM

Commit message: TD1.1 Chages to KIDCAD
Parts:
- added D1, D2, D3, D4: LED, LED_THT:LED_D5.0mm, symbol Device:LED
- added R1, R2, R3, R4: 470, Resistor_THT:R_Axial_DIN0207_L6.3mm_D2.5mm_P10.16mm_Horizontal, symbol Device:R
Connections:
- net GND: now also D1.1 (K), D2.1 (K), D3.1 (K), D4.1 (K)
- net SCL/A5: no longer J2.1 (Pin_1)
- net SDA/A4: no longer J2.2 (Pin_2)
- net *10 renamed LED_D10
- net LED_D10: now also R2.1
- net *11 renamed LED_D11
- net LED_D11: now also R3.1
- net *9 renamed LED_D9
- net LED_D9: now also R1.1
- net 12 renamed LED_D12
- net LED_D12: now also R4.1
- new net: D4.2 (A), R4.2
- new net: D3.2 (A), R3.2
- new net: D1.2 (A), R1.2
- new net: D2.2 (A), R2.2
- new net SCL: J2.1 (Pin_1)
- new net SDA: J2.2 (Pin_2)
- no-connect marks 24 -> 22

Commit message: KICAD modifs
Parts:
- removed D1, D2, D3, D4: LED, LED_THT:LED_D5.0mm, symbol Device:LED
- added C1, C2: C, symbol Device:C
- added LTC1050: ~, symbol LibCapteur:LTC1050
- added R5: R, symbol Device:R
- R1, R2, R3, R4: value 470 -> R; footprint Resistor_THT:R_Axial_DIN0207_L6.3mm_D2.5mm_P10.16mm_Horizontal -> (none)
Connections:
- net LED_D10: no longer R2.1
- net LED_D11: no longer R3.1
- net LED_D12: no longer R4.1
- net LED_D9: no longer R1.1
Other:
- moved on the sheet: J1, J2, J3, J4

Commit message: KICAD MODIFS
Parts:
- added C3, C4: C, symbol Device:C
- added CAP1: ~, symbol LibCapteur:Capteur
- added MP1: ~, Guarrempreintes:MCP41050, symbol Chulo:MPC41050
Connections:
- net +5V: now also LTC1050.7 (V+), C4.1, CAP1.1 (5V)
- net GND: now also C1.2, C2.2, LTC1050.4 (V-), R1.2, R2.2, MP1.4 (VSS)
- net VCC: now also MP1.8 (VCC)
- net at C1.1: now also LTC1050.3 (+IN), R1.1, R2.1, R4.2
- net at C2.1: now also R5.2
- net at R3.1: now also LTC1050.2 (-IN), C3.1
- net at R3.2: now also LTC1050.6 (OUT), R5.1, C3.2
- net at R4.1: now also CAP1.2 (GND)
- no-connect marks 22 -> 25
Other:
- added sheet Amplificateur (ampli.kicad_sch)
- added sheet Modules (Modules.kicad_sch)
- note added: "* Indicates a PWM-capable pin"
- moved on the sheet: C1, C2, R1, R2, R4, R5

Commit message: More kicad modifs
Parts:
- removed MP1: ~, Guarrempreintes:MCP41050, symbol Chulo:MPC41050
- added BT1: ~, symbol LibCapteur:BT_HC-05
- added OLED1, OLED2: ~, symbol LibCapteur:Ecran_OLED
- added ROT1: ~, symbol LibCapteur:EncodRot
- C1, C2, C4: value C -> 100n
- C3: value C -> 1u
- R1, R3: value R -> 100k
- R2, R5: value R -> 1k
- R4: value R -> 10k
Connections:
- net A0 is gone; now on net ADC: J3.1 (Pin_1)
- net GND: now also C4.2
- net ADC: now reaches C2.1, R5.2
- net VCC renamed Vin
Other:
- moved on the sheet: C1

Commit message: Duri
Parts:
- removed BT1: ~, symbol LibCapteur:BT_HC-05
- removed OLED1: ~, symbol LibCapteur:Ecran_OLED
- added BT2: ~, symbol LibCapteur:BT_HC-05
- OLED2: footprint (none) -> LIbCapteurPCB:OLED
Other:
- moved on the sheet: OLED2
Changed lines of the file:
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@@
+	)
+	(symbol
+		(lib_name "BT_HC-05_1")
+		(lib_id "LibCapteur:BT_HC-05")
+		(at 41.91 138.43 0)
+		(unit 1)
+		(exclude_from_sim no)
+		(in_bom yes)
+		(on_board yes)
+		(dnp no)
+		(fields_autoplaced yes)
+		(property "Reference" "BT2"
+			(at 40.64 137.16 0)
+			(effects
+				(font
+					(size 1.27 1.27)
+				)
+			)
+		)
+		(property "Value" "~"
+			(at 40.64 139.7 0)
+			(effects
+				(font
+					(size 1.27 1.27)
+				)
+			)
+		)
+		(property "Footprint" ""
+			(at 41.91 138.43 0)
+			(effects
+				(font
+					(size 1.27 1.27)
+				)
+				(hide yes)
+			)
+		)
+		(property "Datasheet" ""
+			(at 41.91 138.43 0)
+			(effects
+				(font
+					(size 1.27 1.27)
+				)
+				(hide yes)
+			)
+		)
+		(property "Description" ""
+			(at 41.91 138.43 0)
+			(effects
+				(font
+					(size 1.27 1.27)
+				)
+				(hide yes)
+			)
+		)
+		(pin "3"
+		)
+		(pin "2"
+		)
+		(pin "1"
+		)
+		(pin "4"
+		)
+		(instances
+			(project "ProjetCpatKiCad"
+				(path "/e63e39d7-6ac0-4ffd-8aa3-1841a4541b55"
+					(reference "BT2")
+					(unit 1)
+				)
+			)
+		)
 	)
 	(symbol
@@
 	)
 	(symbol
-		(lib_id "LibCapteur:Ecran_OLED")
-		(at 86.36 137.16 0)
-		(unit 1)
-		(exclude_from_sim no)
-		(in_bom yes)
-		(on_board yes)
-		(dnp no)
-		(fields_autoplaced yes)
-		(property "Reference" "OLED1"
-			(at 85.09 135.89 0)
-			(effects
-				(font
-					(size 1.27 1.27)
-				)
-			)
-		)
-		(property "Value" "~"
-			(at 85.09 138.43 0)
-			(effects
-				(font
-					(size 1.27 1.27)
-				)
-			)
-		)
-		(property "Footprint" ""
-			(at 86.36 137.16 0)
-			(effects
-				(font
-					(size 1.27 1.27)
-				)
-				(hide yes)
-			)
-		)
-		(property "Datasheet" ""
-			(at 86.36 137.16 0)
-			(effects
-				(font
-					(size 1.27 1.27)
-				)
-				(hide yes)
-			)
-		)
-		(property "Description" ""
-			(at 86.36 137.16 0)
-			(effects
-				(font
-					(size 1.27 1.27)
-				)
-				(hide yes)
-			)
-		)
-		(pin ""
-		)
-		(pin ""
-		)
-		(pin ""
-		)
-		(pin ""
-		)
-		(instances
-			(project "ProjetCpatKiCad"
-				(path "/e63e39d7-6ac0-4ffd-8aa3-1841a4541b55"
-					(reference "OLED1")
-					(unit 1)
-				)
-			)
-		)
-	)
-	(symbol
 		(lib_id "power:GND")
 		(at 215.9 58.42 0)
@@
 		(lib_name "Ecran_OLED_1")
 		(lib_id "LibCapteur:Ecran_OLED")
-		(at 86.36 160.02 0)
+		(at 83.82 137.16 0)
 		(unit 1)
 		(exclude_from_sim no)
@@
 		(fields_autoplaced yes)
 		(property "Reference" "OLED2"
-			(at 85.09 158.75 0)
+			(at 82.55 135.89 0)
 			(effects
 				(font
@@
 		)
 		(property "Value" "~"
-			(at 85.09 161.29 0)
-			(effects
-				(font
-					(size 1.27 1.27)
-				)
-			)
-		)
-		(property "Footprint" ""
-			(at 86.36 160.02 0)
+			(at 82.55 138.43 0)
+			(effects
+				(font
+					(size 1.27 1.27)
+				)
+			)
+		)
+		(property "Footprint" "LIbCapteurPCB:OLED"
+			(at 83.82 137.16 0)
 			(effects
 				(font
@@
 		)
 		(property "Datasheet" ""
-			(at 86.36 160.02 0)
+			(at 83.82 137.16 0)
 			(effects
 				(font
@@
 		)
 		(property "Description" ""
-			(at 86.36 160.02 0)
+			(at 83.82 137.16 0)
 			(effects
 				(font
@@
 					(unit 1)
 				)
-			)
-		)
-	)
-	(symbol
-		(lib_id "LibCapteur:BT_HC-05")
-		(at 44.45 138.43 0)
-		(unit 1)
-		(exclude_from_sim no)
-		(in_bom yes)
-		(on_board yes)
-		(dnp no)
-		(fields_autoplaced yes)
-		(property "Reference" "BT1"
-			(at 43.18 137.16 0)
-			(effects
-				(font
-					(size 1.27 1.27)
-				)
-			)
-		)
-		(property "Value" "~"
-			(at 43.18 139.7 0)
-			(effects
-				(font
-					(size 1.27 1.27)
-				)
-			)
-		)
-		(property "Footprint" ""
-			(at 44.45 138.43 0)
-			(effects
-				(font
-					(size 1.27 1.27)
-				)
-				(hide yes)
-			)
-		)
-		(property "Datasheet" ""
-			(at 44.45 138.43 0)
-			(effects
-				(font
-					(size 1.27 1.27)
-				)
-				(hide yes)
-			)
-		)
-		(property "Description" ""
-			(at 44.45 138.43 0)
-			(effects
-				(font
-					(size 1.27 1.27)
-				)
-				(hide yes)
-			)
-		)
-		(pin ""
-		)
-		(pin ""
-		)
-		(pin ""
-		)
-		(pin ""
-		)
-		(instances
-			(project "ProjetCpatKiCad"
-				(path "/e63e39d7-6ac0-4ffd-8aa3-1841a4541b55"
-					(reference "BT1")
-					(unit 1)
-				)

Commit message: Modifs
Parts:
- LTC1050: footprint (none) -> LIbCapteurPCB:LTC1050
- renumbered BT2 to BT, OLED2 to OLED, ROT1 to ROT
Changed lines of the file:
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@@
 		(on_board yes)
 		(dnp no)
-		(fields_autoplaced yes)
-		(property "Reference" "BT2"
-			(at 40.64 137.16 0)
+		(property "Reference" "BT"
+			(at 43.942 145.034 0)
 			(effects
 				(font
@@
 			(project "ProjetCpatKiCad"
 				(path "/e63e39d7-6ac0-4ffd-8aa3-1841a4541b55"
-					(reference "BT2")
+					(reference "BT")
 					(unit 1)
 				)
@@
 			)
 		)
-		(property "Footprint" ""
+		(property "Footprint" "LIbCapteurPCB:LTC1050"
 			(at 109.22 55.88 0)
 			(effects
@@
 		(on_board yes)
 		(dnp no)
-		(fields_autoplaced yes)
-		(property "Reference" "OLED2"
-			(at 82.55 135.89 0)
+		(property "Reference" "OLED"
+			(at 87.122 145.288 0)
 			(effects
 				(font
@@
 			(project "ProjetCpatKiCad"
 				(path "/e63e39d7-6ac0-4ffd-8aa3-1841a4541b55"
-					(reference "OLED2")
+					(reference "OLED")
 					(unit 1)
 				)
@@
 		(on_board yes)
 		(dnp no)
-		(fields_autoplaced yes)
-		(property "Reference" "ROT1"
-			(at 138.43 133.35 0)
+		(property "Reference" "ROT"
+			(at 148.59 144.526 0)
 			(effects
 				(font
@@
 			(project "ProjetCpatKiCad"
 				(path "/e63e39d7-6ac0-4ffd-8aa3-1841a4541b55"
-					(reference "ROT1")
-					(unit 1)
-				)
+					(reference "ROT")
+					(unit 1)
+				)
