File: KiCad/ProjetCpatKiCad/ProjetCpatKiCad/ProjetCpatKiCad.kicad_sch (KiCad schematic)
At the start: 19 parts, among them J1 Power, J2 Digital/PWM, J3 Analog, J4 Digital/PWM

Commit message: KICAD final 08/03
Parts:
- added Flex1: ~, symbol LibCapteur:FlexSensor
- LTC1050: footprint LIbCapteurPCB:LTC1050 -> Package_DIP:DIP-8_W7.62mm_LongPads
- renumbered BT to BT1, OLED to OLED1, ROT to ROT1
Changed lines of the file:
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@@
 		(on_board yes)
 		(dnp no)
-		(property "Reference" "BT"
+		(property "Reference" "BT1"
 			(at 43.942 145.034 0)
 			(effects
@@
 			(project "ProjetCpatKiCad"
 				(path "/e63e39d7-6ac0-4ffd-8aa3-1841a4541b55"
-					(reference "BT")
+					(reference "BT1")
 					(unit 1)
 				)
@@
 			)
 		)
-		(property "Footprint" "LIbCapteurPCB:LTC1050"
+		(property "Footprint" "Package_DIP:DIP-8_W7.62mm_LongPads"
 			(at 109.22 55.88 0)
 			(effects
@@
 	)
 	(symbol
+		(lib_id "LibCapteur:FlexSensor")
+		(at 105.41 176.53 0)
+		(unit 1)
+		(exclude_from_sim no)
+		(in_bom yes)
+		(on_board yes)
+		(dnp no)
+		(fields_autoplaced yes)
+		(property "Reference" "Flex1"
+			(at 115.57 175.8949 0)
+			(effects
+				(font
+					(size 1.27 1.27)
+				)
+				(justify left)
+			)
+		)
+		(property "Value" "~"
+			(at 115.57 177.8 0)
+			(effects
+				(font
+					(size 1.27 1.27)
+				)
+				(justify left)
+			)
+		)
+		(property "Footprint" ""
+			(at 105.41 176.53 0)
+			(effects
+				(font
+					(size 1.27 1.27)
+				)
+				(hide yes)
+			)
+		)
+		(property "Datasheet" ""
+			(at 105.41 176.53 0)
+			(effects
+				(font
+					(size 1.27 1.27)
+				)
+				(hide yes)
+			)
+		)
+		(property "Description" ""
+			(at 105.41 176.53 0)
+			(effects
+				(font
+					(size 1.27 1.27)
+				)
+				(hide yes)
+			)
+		)
+		(pin "2"
+		)
+		(pin "1"
+		)
+		(instances
+			(project "ProjetCpatKiCad"
+				(path "/e63e39d7-6ac0-4ffd-8aa3-1841a4541b55"
+					(reference "Flex1")
+					(unit 1)
+				)
+			)
+		)
+	)
+	(symbol
 		(lib_name "Ecran_OLED_1")
 		(lib_id "LibCapteur:Ecran_OLED")
@@
 		(on_board yes)
 		(dnp no)
-		(property "Reference" "OLED"
+		(property "Reference" "OLED1"
 			(at 87.122 145.288 0)
 			(effects
@@
 			(project "ProjetCpatKiCad"
 				(path "/e63e39d7-6ac0-4ffd-8aa3-1841a4541b55"
-					(reference "OLED")
+					(reference "OLED1")
 					(unit 1)
 				)
@@
 		(on_board yes)
 		(dnp no)
-		(property "Reference" "ROT"
+		(property "Reference" "ROT1"
 			(at 148.59 144.526 0)
 			(effects
@@
 			(project "ProjetCpatKiCad"
 				(path "/e63e39d7-6ac0-4ffd-8aa3-1841a4541b55"
-					(reference "ROT")
-					(unit 1)
-				)
+					(reference "ROT1")
+					(unit 1)
+				)

Commit message: Cambios KICAD
Parts:
- BT1: footprint (none) -> LIbCapteurPCB:BT-HC05
- C1, C2, C3, C4: footprint (none) -> Capacitor_SMD:C_0201_0603Metric
- Flex1: footprint (none) -> LIbCapteurPCB:FlexSensor
- MCP1: footprint (none) -> LIbCapteurPCB:DigiPot
- R1, R2, R3, R4, R5: footprint (none) -> Resistor_SMD:R_0201_0603Metric
Changed lines of the file:
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@@
 			)
 		)
-		(property "Footprint" ""
+		(property "Footprint" "Capacitor_SMD:C_0201_0603Metric"
 			(at 67.0052 88.9 0)
 			(effects
@@
 			)
 		)
-		(property "Footprint" ""
+		(property "Footprint" "Capacitor_SMD:C_0201_0603Metric"
 			(at 163.5252 88.9 0)
 			(effects
@@
 			)
 		)
-		(property "Footprint" ""
+		(property "Footprint" "Resistor_SMD:R_0201_0603Metric"
 			(at 84.582 85.09 90)
 			(effects
@@
 			)
 		)
-		(property "Footprint" ""
+		(property "Footprint" "LIbCapteurPCB:DigiPot"
 			(at 143.51 172.72 0)
 			(effects
@@
 			)
 		)
-		(property "Footprint" ""
+		(property "Footprint" "Resistor_SMD:R_0201_0603Metric"
 			(at 141.732 58.42 90)
 			(effects
@@
 			)
 		)
-		(property "Footprint" ""
+		(property "Footprint" "Resistor_SMD:R_0201_0603Metric"
 			(at 75.692 85.09 90)
 			(effects
@@
 			)
 		)
-		(property "Footprint" ""
+		(property "Footprint" "LIbCapteurPCB:BT-HC05"
 			(at 41.91 138.43 0)
 			(effects
@@
 			)
 		)
-		(property "Footprint" ""
+		(property "Footprint" "Resistor_SMD:R_0201_0603Metric"
 			(at 154.94 71.628 90)
 			(effects
@@
 			)
 		)
-		(property "Footprint" ""
+		(property "Footprint" "Capacitor_SMD:C_0201_0603Metric"
 			(at 148.2852 41.91 0)
 			(effects
@@
 			)
 		)
-		(property "Footprint" ""
+		(property "Footprint" "LIbCapteurPCB:FlexSensor"
 			(at 105.41 176.53 0)
 			(effects
@@
 			)
 		)
-		(property "Footprint" ""
+		(property "Footprint" "Resistor_SMD:R_0201_0603Metric"
 			(at 59.69 75.438 90)
 			(effects
@@
 			)
 		)
-		(property "Footprint" ""
+		(property "Footprint" "Capacitor_SMD:C_0201_0603Metric"
 			(at 133.0452 62.23 0)
 			(effects

Commit message: KICAD connections
Connections:
- net *5 is gone; now on net SW: J4.3 (Pin_3)
- net 13 is gone; now on net CLKPOT: J2.5 (Pin_5)
- net 2 is gone; now on net CLK: J4.6 (Pin_6)
- net 4 is gone; now on net DT: J4.4 (Pin_4)
- net 8 is gone; now on net BT_TX: J2.10 (Pin_10)
- net LED_D10 is gone; now on net CS: J2.8 (Pin_8)
- net LED_D11 is gone; now on net SI: J2.7 (Pin_7)
- net LED_D9 is gone; now on net BT_RX: J2.9 (Pin_9)
- net SCL/A5 is gone; now on net SCL: J3.6 (Pin_6)
- net SDA/A4 is gone; now on net SDA: J3.5 (Pin_5)
- net +5V: now also BT1.1 (5V), Flex1.1, MCP1.8 (VCC), OLED1.2 (+5V), ROT1.4 (+5V)
- net A1: now also Flex1.2
- net GND: now also BT1.2 (GND), MCP1.4 (VSS), OLED1.1 (GND), ROT1.5 (GND)
- net SCL: now also OLED1.3 (SCL)
- net SDA: now also OLED1.4 (SDA)
- net CS: now reaches MCP1.1 (CS)
- net CLKPOT: now reaches MCP1.2 (SCK)
- net SI: now reaches MCP1.3 (SI)
- net BT_TX: now reaches BT1.3 (Tx)
- net BT_RX: now reaches BT1.4 (RX)
- net CLK: now reaches ROT1.1 (CLK)
- net DT: now reaches ROT1.2 (DATA)
- net SW: now reaches ROT1.3 (SWITCH)
- net LED_D12 renamed 12
- no-connect marks 25 -> 18
Other:
- title: Démo Shield Arduino -> Shield Arduino UNO projet

Commit message: Añadidos librerias KICAD
Connections:
- net +5V: no longer MCP1.8 (VCC)
- net A1: no longer Flex1.2
- net GND: now also Flex1.2; no longer MCP1.4 (VSS)
- net SCL: no longer J3.6 (Pin_6), OLED1.3 (SCL)
- net SDA: no longer J3.5 (Pin_5), OLED1.4 (SDA)
- net BT_RX: no longer names the net of BT1.4 (RX)
- net BT_RX: no longer J2.9 (Pin_9)
- net BT_TX: no longer names the net of BT1.3 (Tx)
- net BT_TX: no longer J2.10 (Pin_10)
- net CLK: no longer names the net of ROT1.1 (CLK)
- net CLK: no longer J4.6 (Pin_6)
- net CLKPOT: no longer names the net of MCP1.2 (SCK)
- net CLKPOT: no longer J2.5 (Pin_5)
- net CS: no longer names the net of MCP1.1 (CS)
- net CS: no longer J2.8 (Pin_8)
- net DT: no longer names the net of ROT1.2 (DATA)
- net DT: no longer J4.4 (Pin_4)
- net SI: no longer names the net of MCP1.3 (SI)
- net SI: no longer J2.7 (Pin_7)
- net SW: no longer names the net of ROT1.3 (SWITCH)
- net SW: no longer J4.3 (Pin_3)
- new net *10: J2.8 (Pin_8)
- new net *11: J2.7 (Pin_7)
- new net *5: J4.3 (Pin_3)
- new net *9: J2.9 (Pin_9)
- new net 13: J2.5 (Pin_5)
- new net 2: J4.6 (Pin_6)
- new net 4: J4.4 (Pin_4)
- new net 8: J2.10 (Pin_10)
- new net SCL/A5: J3.6 (Pin_6)
- new net SDA/A4: J3.5 (Pin_5)
- no-connect marks 18 -> 25
Other:
- title: Shield Arduino UNO projet -> Démo Shield Arduino

Commit message: Footprints and schematics
Parts:
- CAP1: footprint (none) -> LIbCapteurPCB:Capteur Gaz
- ROT1: footprint (none) -> LIbCapteurPCB:ROT
Connections:
- net *10 is gone; now on net M-1: CS: J2.8 (Pin_8)
- net *5 is gone; now on net R-3: SWITCH: J4.3 (Pin_3)
- net *9 is gone; now on net B-4: Rx: J2.9 (Pin_9)
- net 2 is gone; now on net R-1: CLK: J4.6 (Pin_6)
- net 4 is gone; now on net R-2: DATA: J4.4 (Pin_4)
- net 8 is gone; now on net B-3: Tx: J2.10 (Pin_10)
- net SCL/A5 is gone; now on net O-3: SCL: J3.6 (Pin_6)
- net SDA/A4 is gone; now on net O-4: SDA: J3.5 (Pin_5)
- net +5V: now also MCP1.8 (VCC)
- net GND: now also MCP1.4 (VSS); no longer Flex1.2
- net M-1: CS: now reaches MCP1.1 (CS)
- net M-2: SCK: now reaches MCP1.2 (SCK)
- net M-3: SI: now reaches MCP1.3 (SI)
- net M-5: A: now reaches MCP1.5 (A)
- net M-6: W: now reaches MCP1.6 (W)
- net M-7: B: now reaches MCP1.7 (B)
- net B-3: Tx: now reaches BT1.3 (Tx)
- net B-4: Rx: now reaches BT1.4 (RX)
- net O-3: SCL: now reaches OLED1.3 (SCL)
- net O-4: SDA: now reaches OLED1.4 (SDA)
- net R-1: CLK: now reaches ROT1.1 (CLK)
- net R-2: DATA: now reaches ROT1.2 (DATA)
- net R-3: SWITCH: now reaches ROT1.3 (SWITCH)
- net A1 renamed F-2
- net F-2: now also Flex1.2
- no-connect marks 25 -> 20
Other:
- moved on the sheet: Flex1

Commit message: un poquito de pcb
Parts:
- Flex1: footprint LIbCapteurPCB:FlexSensor -> LIbCapteurPCB:F_SENSE
- LTC1050: footprint Package_DIP:DIP-8_W7.62mm_LongPads -> LIbCapteurPCB:LTC1050
Changed lines of the file:
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@@
 			)
 		)
-		(property "Footprint" "Package_DIP:DIP-8_W7.62mm_LongPads"
+		(property "Footprint" "LIbCapteurPCB:LTC1050"
 			(at 109.22 55.88 0)
 			(effects
@@
 			)
 		)
-		(property "Footprint" "LIbCapteurPCB:FlexSensor"
+		(property "Footprint" "LIbCapteurPCB:F_SENSE"
 			(at 58.42 176.53 0)
 			(effects

Commit message: tiqui
Parts:
- C1, C2, C3: footprint Capacitor_SMD:C_0201_0603Metric -> Capacitor_THT:C_Axial_L3.8mm_D2.6mm_P7.50mm_Horizontal
- C4: footprint Capacitor_SMD:C_0201_0603Metric -> Capacitor_THT:C_Rect_L4.6mm_W5.5mm_P2.50mm_MKS02_FKP02
- R1, R2, R3, R4, R5: footprint Resistor_SMD:R_0201_0603Metric -> Resistor_THT:R_Axial_DIN0204_L3.6mm_D1.6mm_P1.90mm_Vertical
Connections:
- net *11 is gone; now on net M-3: SI: J2.7 (Pin_7)
- net 13 is gone; now on net M-2: SCK: J2.5 (Pin_5)
- net +5V: no longer MCP1.8 (VCC)
- net ADC: now also J3.2 (Pin_2); no longer J3.1 (Pin_1)
- net F-2: now also J3.1 (Pin_1); no longer J3.2 (Pin_2)
- net GND: no longer MCP1.4 (VSS)
Changed lines of the file:
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@@
 	)
 	(no_connect
+		(at 153.67 168.91)
+	)
+	(no_connect
 		(at 203.2 43.18)
 	)
@@
 	)
 	(no_connect
-		(at 205.74 73.66)
+		(at 132.08 180.34)
 	)
 	(no_connect
-		(at 120.65 57.15)
+		(at 205.74 73.66)
 	)
 	(no_connect
-		(at 262.89 48.26)
+		(at 120.65 57.15)
 	)
 	(no_connect
@@
 	)
 	(no_connect
-		(at 259.08 43.18)
-	)
-	(no_connect
 		(at 218.44 38.1)
 	)
@@
 	(wire
 		(pts
-			(xy 246.38 50.8) (xy 262.89 50.8)
-		)
-		(stroke
-			(width 0)
-			(type solid)
-		)
-	)
-	(wire
-		(pts
 			(xy 143.51 54.61) (xy 143.51 50.8)
 		)
@@
 	(wire
 		(pts
+			(xy 246.38 50.8) (xy 262.89 50.8)
+		)
+		(stroke
+			(width 0)
+			(type default)
+		)
+	)
+	(wire
+		(pts
 			(xy 246.38 76.2) (xy 259.08 76.2)
 		)
@@
 	(wire
 		(pts
-			(xy 246.38 43.18) (xy 259.08 43.18)
+			(xy 246.38 43.18) (xy 262.89 43.18)
 		)
 		(stroke
@@
 	(global_label "F-2"
 		(shape input)
-		(at 203.2 68.58 180)
+		(at 203.2 66.04 180)
 		(fields_autoplaced yes)
 		(effects
@@
 		)
 		(property "Intersheetrefs" "${INTERSHEET_REFS}"
-			(at 196.2492 68.58 0)
+			(at 196.2492 66.04 0)
 			(effects
 				(font
@@
 		)
 	)
+	(global_label "M-3: SI"
+		(shape input)
+		(at 262.89 48.26 0)
+		(fields_autoplaced yes)
+		(effects
+			(font
+				(size 1.27 1.27)
+			)
+			(justify left)
+		)
+		(property "Intersheetrefs" "${INTERSHEET_REFS}"
+			(at 273.5903 48.26 0)
+			(effects
+				(font
+					(size 1.27 1.27)
+				)
+				(justify left)
+				(hide yes)
+			)
+		)
+	)
 	(global_label "B-4: Rx"
 		(shape input)
@@
 	(global_label "ADC"
 		(shape input)
-		(at 203.2 66.04 180)
+		(at 203.2 68.58 180)
 		(fields_autoplaced yes)
 		(effects
@@
 		)
 		(property "Intersheetrefs" "${INTERSHEET_REFS}"
-			(at 196.4911 66.04 0)
+			(at 196.4911 68.58 0)
 			(effects
 				(font
@@
 	(global_label "M-2: SCK"
 		(shape input)
+		(at 262.89 43.18 0)
+		(fields_autoplaced yes)
+		(effects
+			(font
+				(size 1.27 1.27)
+			)
+			(justify left)
+		)
+		(property "Intersheetrefs" "${INTERSHEET_REFS}"
+			(at 275.5255 43.18 0)
+			(effects
+				(font
+					(size 1.27 1.27)
+				)
+				(justify left)
+				(hide yes)
+			)
+		)
+	)
+	(global_label "M-2: SCK"
+		(shape input)
 		(at 132.08 172.72 180)
 		(fields_autoplaced yes)
@@
 			)
 		)
-		(property "Footprint" "Capacitor_SMD:C_0201_0603Metric"
+		(property "Footprint" "Capacitor_THT:C_Axial_L3.8mm_D2.6mm_P7.50mm_Horizontal"
 			(at 67.0052 88.9 0)
 			(effects
@@
 			)
 		)
-		(property "Footprint" "Capacitor_SMD:C_0201_0603Metric"
+		(property "Footprint" "Capacitor_THT:C_Axial_L3.8mm_D2.6mm_P7.50mm_Horizontal"
 			(at 163.5252 88.9 0)
 			(effects
@@
 			)
 		)
-		(property "Footprint" "Resistor_SMD:R_0201_0603Metric"
+		(property "Footprint" "Resistor_THT:R_Axial_DIN0204_L3.6mm_D1.6mm_P1.90mm_Vertical"
 			(at 84.582 85.09 90)
 			(effects
@@
 			)
 		)
-		(property "Footprint" "Resistor_SMD:R_0201_0603Metric"
+		(property "Footprint" "Resistor_THT:R_Axial_DIN0204_L3.6mm_D1.6mm_P1.90mm_Vertical"
 			(at 141.732 58.42 90)
 			(effects
@@
 			)
 		)
-		(property "Footprint" "Resistor_SMD:R_0201_0603Metric"
+		(property "Footprint" "Resistor_THT:R_Axial_DIN0204_L3.6mm_D1.6mm_P1.90mm_Vertical"
 			(at 75.692 85.09 90)
 			(effects
@@
 			)
 		)
-		(property "Footprint" "Resistor_SMD:R_0201_0603Metric"
+		(property "Footprint" "Resistor_THT:R_Axial_DIN0204_L3.6mm_D1.6mm_P1.90mm_Vertical"
 			(at 154.94 71.628 90)
 			(effects
@@
 	)
 	(symbol
-		(lib_id "power:+5V")
-		(at 153.67 168.91 270)
-		(unit 1)
-		(exclude_from_sim no)
-		(in_bom yes)
-		(on_board yes)
-		(dnp no)
-		(property "Reference" "#PWR020"
-			(at 149.86 168.91 0)
-			(effects
-				(font
-					(size 1.27 1.27)
-				)
-				(hide yes)
-			)
-		)
-		(property "Value" "+5V"
-			(at 156.718 169.2656 90)
-			(effects
-				(font
-					(size 1.27 1.27)
-				)
-				(justify left)
-			)
-		)
-		(property "Footprint" ""
-			(at 153.67 168.91 0)
-			(effects
-				(font
-					(size 1.27 1.27)
-				)
-			)
-		)
-		(property "Datasheet" ""
-			(at 153.67 168.91 0)
-			(effects
-				(font
-					(size 1.27 1.27)
-				)
-			)
-		)
-		(property "Description" "Power symbol creates a global label with name \"+5V\""
-			(at 153.67 168.91 0)
-			(effects
-				(font
-					(size 1.27 1.27)
-				)
-				(hide yes)
-			)
-		)
-		(pin "1"
-		)
-		(instances
-			(project "ProjetCpatKiCad"
-				(path "/e63e39d7-6ac0-4ffd-8aa3-1841a4541b55"
-					(reference "#PWR020")
-					(unit 1)
-				)
-			)
-		)
-	)
-	(symbol
 		(lib_id "power:GND")
 		(at 67.31 140.97 270)
@@
 			)
 		)
-		(property "Footprint" "Capacitor_SMD:C_0201_0603Metric"
+		(property "Footprint" "Capacitor_THT:C_Rect_L4.6mm_W5.5mm_P2.50mm_MKS02_FKP02"
 			(at 148.2852 41.91 0)
 			(effects
@@
 			)
 		)
-		(property "Footprint" "Resistor_SMD:R_0201_0603Metric"
+		(property "Footprint" "Resistor_THT:R_Axial_DIN0204_L3.6mm_D1.6mm_P1.90mm_Vertical"
 			(at 59.69 75.438 90)
 			(effects
@@
 	(symbol
 		(lib_id "power:GND")
-		(at 132.08 180.34 270)
-		(unit 1)
-		(exclude_from_sim no)
-		(in_bom yes)
-		(on_board yes)
-		(dnp no)
-		(property "Reference" "#PWR021"
-			(at 125.73 180.34 0)
-			(effects
-				(font
-					(size 1.27 1.27)
-				)
-				(hide yes)
-			)
-		)
-		(property "Value" "GND"
-			(at 128.27 180.34 0)
-			(effects
-				(font
-					(size 1.27 1.27)
-				)
-			)
-		)
-		(property "Footprint" ""
-			(at 132.08 180.34 0)
-			(effects
-				(font
-					(size 1.27 1.27)
-				)
-			)
-		)
-		(property "Datasheet" ""
-			(at 132.08 180.34 0)
-			(effects
-				(font
-					(size 1.27 1.27)
-				)
-			)
-		)
-		(property "Description" "Power symbol creates a global label with name \"GND\" , ground"
-			(at 132.08 180.34 0)
-			(effects
-				(font
-					(size 1.27 1.27)
-				)
-				(hide yes)
-			)
-		)
-		(pin "1"
-		)
-		(instances
-			(project "ProjetCpatKiCad"
-				(path "/e63e39d7-6ac0-4ffd-8aa3-1841a4541b55"
-					(reference "#PWR021")
-					(unit 1)
-				)
-			)
-		)
-	)
-	(symbol
-		(lib_id "power:GND")
 		(at 107.95 109.22 0)
 		(unit 1)
@@
 			)
 		)
-		(property "Footprint" "Capacitor_SMD:C_0201_0603Metric"
+		(property "Footprint" "Capacitor_THT:C_Axial_L3.8mm_D2.6mm_P7.50mm_Horizontal"
 			(at 133.0452 62.23 0)
 			(effects
