File: KiCad/ProjetCpatKiCad/ProjetCpatKiCad/ProjetCpatKiCad.kicad_sch (KiCad schematic)
At the start: 19 parts, among them J1 Power, J2 Digital/PWM, J3 Analog, J4 Digital/PWM

Commit message: Kicad modelos 3d
Changed lines of the file:
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@@
 	)
 	(junction
-		(at 86.36 104.14)
-		(diameter 0)
-		(color 0 0 0 0)
-	)
-	(junction
 		(at 77.47 73.66)
 		(diameter 0)
@@
 	(wire
 		(pts
-			(xy 86.36 88.9) (xy 86.36 104.14)
-		)
-		(stroke
-			(width 0)
-			(type default)
-		)
-	)
-	(wire
-		(pts
 			(xy 215.9 50.8) (xy 215.9 53.34)
 		)
@@
 	(wire
 		(pts
-			(xy 107.95 104.14) (xy 86.36 104.14)
-		)
-		(stroke
-			(width 0)
-			(type default)
-		)
-	)
-	(wire
-		(pts
 			(xy 246.38 68.58) (xy 259.08 68.58)
 		)
@@
 	(wire
 		(pts
+			(xy 246.38 55.88) (xy 262.89 55.88)
+		)
+		(stroke
+			(width 0)
+			(type default)
+		)
+	)
+	(wire
+		(pts
 			(xy 86.36 73.66) (xy 93.98 73.66)
 		)
@@
 	(wire
 		(pts
-			(xy 86.36 104.14) (xy 77.47 104.14)
+			(xy 77.47 104.14) (xy 107.95 104.14)
 		)
 		(stroke
@@
 		)
 	)
-	(wire
-		(pts
-			(xy 246.38 55.88) (xy 262.89 55.88)
-		)
-		(stroke
-			(width 0)
-			(type solid)
-		)
-	)
 	(text "* Indicates a PWM-capable pin"
 		(exclude_from_sim no)
@@
 		)
 	)
-	(global_label "M-6: W"
-		(shape input)
-		(at 86.36 88.9 0)
-		(fields_autoplaced yes)
-		(effects
-			(font
-				(size 1.27 1.27)
-			)
-			(justify left)
-		)
-		(property "Intersheetrefs" "${INTERSHEET_REFS}"
-			(at 96.6974 88.9 0)
-			(effects
-				(font
-					(size 1.27 1.27)
-				)
-				(justify left)
-				(hide yes)
-			)
-		)
-	)
 	(global_label "O-4: SDA"
 		(shape input)
@@
 		)
 	)
-	(global_label "M-6: W"
-		(shape input)
-		(at 153.67 176.53 0)
-		(fields_autoplaced yes)
-		(effects
-			(font
-				(size 1.27 1.27)
-			)
-			(justify left)
-		)
-		(property "Intersheetrefs" "${INTERSHEET_REFS}"
-			(at 164.0074 176.53 0)
-			(effects
-				(font
-					(size 1.27 1.27)
-				)
-				(justify left)
-				(hide yes)
-			)
-		)
-	)
 	(global_label "M-7: B"
 		(shape input)
@@
 					(unit 1)
 				)
+			)
+		)
+	)
+	(symbol
+		(lib_id "power:GND")
+		(at 153.67 176.53 90)
+		(unit 1)
+		(exclude_from_sim no)
+		(in_bom yes)
+		(on_board yes)
+		(dnp no)
+		(property "Reference" "#PWR019"
+			(at 160.02 176.53 0)
+			(effects
+				(font
+					(size 1.27 1.27)
+				)
+				(hide yes)
+			)
+		)
+		(property "Value" "GND"
+			(at 157.48 176.53 0)
+			(effects
+				(font
+					(size 1.27 1.27)
+				)
+			)
+		)
+		(property "Footprint" ""
+			(at 153.67 176.53 0)
+			(effects
+				(font
+					(size 1.27 1.27)
+				)
+			)
+		)
+		(property "Datasheet" ""
+			(at 153.67 176.53 0)
+			(effects
+				(font
+					(size 1.27 1.27)
+				)
+			)
+		)
+		(property "Description" "Power symbol creates a global label with name \"GND\" , ground"
+			(at 153.67 176.53 0)
+			(effects
+				(font
+					(size 1.27 1.27)
+				)
+				(hide yes)
+			)
+		)
+		(pin "1"
+		)
+		(instances
+			(project "ProjetCpatKiCad"
+				(path "/e63e39d7-6ac0-4ffd-8aa3-1841a4541b55"
+					(reference "#PWR019")
+					(unit 1)
+				)

Commit message: Kicad con servo
Parts:
- added SV1: ~, ChuloPCB:SIP-3, symbol Chulo:Servo
Connections:
- net +5V: now also SV1.2 (VCC)
- net GND: now also SV1.3 (GND)
- net *6 renamed Dig
- net Dig: now also SV1.1 (Dig)
- no-connect marks 20 -> 19
