File: KiCad/ProjetCpatKiCad/ProjetCpatKiCad/ProjetCpatKiCad.kicad_pcb (KiCad board)
At the start: 2 copper layers, 68.6 x 53.3 mm, 8 parts, among them J1 Power, J2 Digital/PWM, J3 Analog, J4 Digital/PWM

Commit message: TD1.1 Chages to KIDCAD
Parts:
- added D1: LED, LED_THT:LED_D5.0mm, F.Cu at (148.0, 61.0)
- added D2: LED, LED_THT:LED_D5.0mm, F.Cu at (148.0, 69.0)
- added D3: LED, LED_THT:LED_D5.0mm, F.Cu at (148.0, 76.5)
- added D4: LED, LED_THT:LED_D5.0mm, F.Cu at (148.0, 84.0)
- added R1: 470, Resistor_THT:R_Axial_DIN0207_L6.3mm_D2.5mm_P10.16mm_Horizontal, F.Cu at (142.2, 68.1)
- added R2: 470, Resistor_THT:R_Axial_DIN0207_L6.3mm_D2.5mm_P10.16mm_Horizontal, F.Cu at (138.2, 68.1)
- added R3: 470, Resistor_THT:R_Axial_DIN0207_L6.3mm_D2.5mm_P10.16mm_Horizontal, F.Cu at (134.1, 68.1)
- added R4: 470, Resistor_THT:R_Axial_DIN0207_L6.3mm_D2.5mm_P10.16mm_Horizontal, F.Cu at (130.1, 68.1)
Connections:
- J2 pad 1: /SCL/A5 -> /SCL
- J2 pad 2: /SDA/A4 -> /SDA
- J2 pad 6: /12 -> /LED_D12
- J2 pad 7: /*11 -> /LED_D11
- J2 pad 8: /*10 -> /LED_D10
- J2 pad 9: /*9 -> /LED_D9

Commit message: Duri
Parts:
- removed D1, D2, D3, D4: LED, LED_THT:LED_D5.0mm
- removed R1, R2, R3, R4: 470, Resistor_THT:R_Axial_DIN0207_L6.3mm_D2.5mm_P10.16mm_Horizontal

Commit message: more
Other:
- board text added: "delcampo@insa-toulouse.fr"
Changed lines of the file:
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@@
 		(layer "Edge.Cuts")
+	)
+	(gr_text "delcampo@insa-toulouse.fr\n"
+		(at 104 58.5 90)
+		(layer "B.Cu")
+		(effects
+			(font
+				(size 1.5 1.5)
+				(thickness 0.3)
+				(bold yes)
+			)
+			(justify left bottom mirror)
+		)
 	)
 	(gr_text "ICSP"

Commit message: kicad
Parts:
- added LTC1050: ~, LIbCapteurPCB:LTC1050, F.Cu at (132.7, 69.4)
- added OLED1: ~, LIbCapteurPCB:OLED, F.Cu at (132.7, 77.2)
Connections:
- net /A0 renamed ADC
- net VCC renamed /Vin

Commit message: KICAD final 08/03
Parts:
- LTC1050: footprint LIbCapteurPCB:LTC1050 -> Package_DIP:DIP-8_W7.62mm_LongPads
- moved OLED1 13.8 mm to (138.5, 64.7)
- moved LTC1050 5.25 mm to (130.8, 74.2)
Routing:
- added copper zone on B.Cu, net GND

Commit message: Cambios KICAD
Parts:
- added BT1: ~, LIbCapteurPCB:BT-HC05, F.Cu at (112.7, 70.7)
- added C1: 100n, Capacitor_SMD:C_0201_0603Metric, F.Cu at (119.8, 69.0)
- added C2: 100n, Capacitor_SMD:C_0201_0603Metric, F.Cu at (119.8, 70.8)
- added C3: 1u, Capacitor_SMD:C_0201_0603Metric, F.Cu at (119.8, 72.5)
- added C4: 100n, Capacitor_SMD:C_0201_0603Metric, F.Cu at (122.2, 69.0)
- added Flex1: ~, LIbCapteurPCB:FlexSensor, F.Cu at (120.6, 62.3)
- added MCP1: ~, LIbCapteurPCB:DigiPot, F.Cu at (112.7, 62.6)
- added R1: 100k, Resistor_SMD:R_0201_0603Metric, F.Cu at (122.2, 70.8)
- added R2: 1k, Resistor_SMD:R_0201_0603Metric, F.Cu at (122.2, 72.5)
- added R3: 100k, Resistor_SMD:R_0201_0603Metric, F.Cu at (124.7, 69.0)
- added R4: 10k, Resistor_SMD:R_0201_0603Metric, F.Cu at (124.7, 70.8)
- added R5: 1k, Resistor_SMD:R_0201_0603Metric, F.Cu at (124.7, 72.5)

Commit message: KICAD connections
Parts:
- moved MCP1 41.0 mm to (153.7, 62.6), turned to -90 degrees
- moved OLED1 28.4 mm to (165.0, 75.0), turned to 90 degrees
- moved BT1 26.0 mm to (135.0, 57.5)
- moved Flex1 15.0 mm to (107.5, 55.0)
- moved LTC1050 7.25 mm to (128.7, 81.2)
Changed lines of the file:
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@@
 	(footprint "LIbCapteurPCB:BT-HC05"
 		(layer "F.Cu")
-		(at 112.66 70.725)
+		(at 135 57.5)
 		(property "Reference" "BT1"
 			(at 0 2.5 0)
@@
 	(footprint "LIbCapteurPCB:OLED"
 		(layer "F.Cu")
-		(at 138.525 64.745)
+		(at 165 75 90)
 		(property "Reference" "OLED1"
-			(at 0 2.5 0)
+			(at 0 2.5 90)
 			(unlocked yes)
 			(layer "F.SilkS")
@@
 		)
 		(property "Value" "~"
-			(at 0 -2.5 0)
+			(at 0 -2.5 90)
 			(unlocked yes)
 			(layer "F.Fab")
@@
 		)
 		(property "Footprint" "LIbCapteurPCB:OLED"
-			(at 0 0 0)
+			(at 0 0 90)
 			(unlocked yes)
 			(layer "F.Fab")
@@
 		)
 		(property "Datasheet" ""
-			(at 0 0 0)
+			(at 0 0 90)
 			(unlocked yes)
 			(layer "F.Fab")
@@
 		)
 		(property "Description" ""
-			(at 0 0 0)
+			(at 0 0 90)
 			(unlocked yes)
 			(layer "F.Fab")
@@
 		(attr through_hole)
 		(fp_line
+			(start 5.31 -1.5)
+			(end 5.31 1.5)
+			(stroke
+				(width 0.12)
+				(type default)
+			)
+			(layer "F.SilkS")
+		)
+		(fp_line
+			(start -2.54 -1.5)
+			(end -2.54 1.5)
+			(stroke
+				(width 0.12)
+				(type default)
+			)
+			(layer "F.SilkS")
+		)
+		(fp_line
 			(start -5.31 -1.5)
 			(end 5.31 -1.5)
@@
 		)
 		(fp_line
+			(start 5.31 1.5)
+			(end -5.31 1.5)
+			(stroke
+				(width 0.12)
+				(type default)
+			)
+			(layer "F.SilkS")
+		)
+		(fp_line
 			(start -5.31 1.5)
 			(end -5.31 -1.5)
@@
 		)
 		(fp_line
-			(start -2.54 -1.5)
-			(end -2.54 1.5)
-			(stroke
-				(width 0.12)
-				(type default)
-			)
-			(layer "F.SilkS")
-		)
-		(fp_line
-			(start 5.31 -1.5)
-			(end 5.31 1.5)
-			(stroke
-				(width 0.12)
-				(type default)
-			)
-			(layer "F.SilkS")
-		)
-		(fp_line
-			(start 5.31 1.5)
-			(end -5.31 1.5)
-			(stroke
-				(width 0.12)
-				(type default)
-			)
-			(layer "F.SilkS")
+			(start 5.06 -1.25)
+			(end 5.06 1.25)
+			(stroke
+				(width 0.05)
+				(type default)
+			)
+			(layer "F.CrtYd")
 		)
 		(fp_line
@@
 		)
 		(fp_line
+			(start 5.06 1.25)
+			(end -5.06 1.25)
+			(stroke
+				(width 0.05)
+				(type default)
+			)
+			(layer "F.CrtYd")
+		)
+		(fp_line
 			(start -5.06 1.25)
 			(end -5.06 -1.25)
@@
 			(layer "F.CrtYd")
 		)
-		(fp_line
-			(start 5.06 -1.25)
-			(end 5.06 1.25)
-			(stroke
-				(width 0.05)
-				(type default)
-			)
-			(layer "F.CrtYd")
-		)
-		(fp_line
-			(start 5.06 1.25)
-			(end -5.06 1.25)
-			(stroke
-				(width 0.05)
-				(type default)
-			)
-			(layer "F.CrtYd")
-		)
 		(pad "1" thru_hole rect
-			(at -3.81 0)
+			(at -3.81 0 90)
 			(size 2 2.54)
 			(drill 1)
@@
 		)
 		(pad "2" thru_hole oval
-			(at -1.27 0)
+			(at -1.27 0 90)
 			(size 2 2.54)
 			(drill 1)
@@
 		)
 		(pad "3" thru_hole oval
-			(at 1.27 0)
+			(at 1.27 0 90)
 			(size 2 2.54)
 			(drill 1)
@@
 		)
 		(pad "4" thru_hole oval
-			(at 3.81 0)
+			(at 3.81 0 90)
 			(size 2 2.54)
 			(drill 1)
@@
 	(footprint "LIbCapteurPCB:FlexSensor"
 		(layer "F.Cu")
-		(at 120.59 62.305)
+		(at 107.5 55)
 		(property "Reference" "Flex1"
 			(at -2.5 0 90)
@@
 	(footprint "LIbCapteurPCB:DigiPot"
 		(layer "F.Cu")
-		(at 112.66 62.575)
+		(at 153.69 62.575 -90)
 		(property "Reference" "MCP1"
-			(at -6.31 0 90)
+			(at -6.31 0 0)
 			(unlocked yes)
 			(layer "F.SilkS")
@@
 		)
 		(property "Value" "~"
-			(at 0 0 0)
+			(at 0 0 -90)
 			(unlocked yes)
 			(layer "F.Fab")
@@
 		)
 		(property "Footprint" "LIbCapteurPCB:DigiPot"
-			(at 0 0 0)
+			(at 0 0 -90)
 			(unlocked yes)
 			(layer "F.Fab")
@@
 		)
 		(property "Datasheet" ""
-			(at 0 0 0)
+			(at 0 0 -90)
 			(unlocked yes)
 			(layer "F.Fab")
@@
 		)
 		(property "Description" ""
-			(at 0 0 0)
+			(at 0 0 -90)
 			(unlocked yes)
 			(layer "F.Fab")
@@
 		(attr through_hole)
 		(fp_line
+			(start -5.31 5.53)
+			(end 5.31 5.53)
+			(stroke
+				(width 0.12)
+				(type default)
+			)
+			(layer "F.SilkS")
+		)
+		(fp_line
+			(start 5.31 5.53)
+			(end 5.31 -5.53)
+			(stroke
+				(width 0.12)
+				(type default)
+			)
+			(layer "F.SilkS")
+		)
+		(fp_line
+			(start -5.31 1.843333)
+			(end -5.31 5.53)
+			(stroke
+				(width 0.12)
+				(type default)
+			)
+			(layer "F.SilkS")
+		)
+		(fp_line
+			(start -4.95 1.843333)
+			(end -5.31 1.843333)
+			(stroke
+				(width 0.12)
+				(type default)
+			)
+			(layer "F.SilkS")
+		)
+		(fp_line
+			(start -5.31 -1.843333)
+			(end -4.95 -1.843333)
+			(stroke
+				(width 0.12)
+				(type default)
+			)
+			(layer "F.SilkS")
+		)
+		(fp_line
+			(start -4.95 -1.843333)
+			(end -4.95 1.843333)
+			(stroke
+				(width 0.12)
+				(type default)
+			)
+			(layer "F.SilkS")
+		)
+		(fp_line
 			(start -5.31 -5.53)
 			(end -5.31 -1.843333)
@@
 		)
 		(fp_line
-			(start -5.31 -1.843333)
-			(end -4.95 -1.843333)
-			(stroke
-				(width 0.12)
-				(type default)
-			)
-			(layer "F.SilkS")
-		)
-		(fp_line
-			(start -5.31 1.843333)
-			(end -5.31 5.53)
-			(stroke
-				(width 0.12)
-				(type default)
-			)
-			(layer "F.SilkS")
-		)
-		(fp_line
-			(start -5.31 5.53)
-			(end 5.31 5.53)
-			(stroke
-				(width 0.12)
-				(type default)
-			)
-			(layer "F.SilkS")
-		)
-		(fp_line
-			(start -4.95 -1.843333)
-			(end -4.95 1.843333)
-			(stroke
-				(width 0.12)
-				(type default)
-			)
-			(layer "F.SilkS")
-		)
-		(fp_line
-			(start -4.95 1.843333)
-			(end -5.31 1.843333)
-			(stroke
-				(width 0.12)
-				(type default)
-			)
-			(layer "F.SilkS")
-		)
-		(fp_line
 			(start 5.31 -5.53)
 			(end -5.31 -5.53)
@@
 		)
 		(fp_line
-			(start 5.31 5.53)
-			(end 5.31 -5.53)
-			(stroke
-				(width 0.12)
-				(type default)
-			)
-			(layer "F.SilkS")
+			(start -5.06 5.28)
+			(end -5.06 -5.28)
+			(stroke
+				(width 0.05)
+				(type default)
+			)
+			(layer "F.CrtYd")
+		)
+		(fp_line
+			(start 5.06 5.28)
+			(end -5.06 5.28)
+			(stroke
+				(width 0.05)
+				(type default)
+			)
+			(layer "F.CrtYd")
 		)
 		(fp_line
@@
 		)
 		(fp_line
-			(start -5.06 5.28)
-			(end -5.06 -5.28)
-			(stroke
-				(width 0.05)
-				(type default)
-			)
-			(layer "F.CrtYd")
-		)
-		(fp_line
 			(start 5.06 -5.28)
 			(end 5.06 5.28)
@@
 			(layer "F.CrtYd")
 		)
-		(fp_line
-			(start 5.06 5.28)
-			(end -5.06 5.28)
-			(stroke
-				(width 0.05)
-				(type default)
-			)
-			(layer "F.CrtYd")
-		)
 		(pad "1" thru_hole rect
-			(at -3.81 3.76)
+			(at -3.81 3.76 270)
 			(size 2 2.54)
 			(drill 1)
@@
 		)
 		(pad "2" thru_hole oval
-			(at -1.27 3.76)
+			(at -1.27 3.76 270)
 			(size 2 2.54)
 			(drill 1)
@@
 		)
 		(pad "3" thru_hole oval
-			(at 1.27 3.76)
+			(at 1.27 3.76 270)
 			(size 2 2.54)
 			(drill 1)
@@
 		)
 		(pad "4" thru_hole oval
-			(at 3.81 3.76)
+			(at 3.81 3.76 270)
 			(size 2 2.54)
 			(drill 1)
@@
 		)
 		(pad "5" thru_hole oval
-			(at 3.81 -3.76)
+			(at 3.81 -3.76 270)
 			(size 2 2.54)
 			(drill 1)
@@
 		)
 		(pad "6" thru_hole oval
-			(at 1.27 -3.76)
+			(at 1.27 -3.76 270)
 			(size 2 2.54)
 			(drill 1)
@@
 		)
 		(pad "7" thru_hole oval
-			(at -1.27 -3.76)
+			(at -1.27 -3.76 270)
 			(size 2 2.54)
 			(drill 1)
@@
 		)
 		(pad "8" thru_hole oval
-			(at -3.81 -3.76)
+			(at -3.81 -3.76 270)
 			(size 2 2.54)
 			(drill 1)
@@
 	(footprint "Package_DIP:DIP-8_W7.62mm_LongPads"
 		(layer "F.Cu")
-		(at 130.75 74.25)
+		(at 128.675 81.2)
 		(descr "8-lead though-hole mounted DIP package, row spacing 7.62 mm (300 mils), LongPads")
 		(tags "THT DIP DIL PDIP 2.54mm 7.62mm 300mil LongPads")

Commit message: un poquito de pcb
Parts:
- added CAP1: ~, LIbCapteurPCB:Capteur Gaz, F.Cu at (113.5, 66.5)
- added ROT1: ~, LIbCapteurPCB:ROT, F.Cu at (155.0, 58.0)
- Flex1: footprint LIbCapteurPCB:FlexSensor -> LIbCapteurPCB:F_SENSE
- LTC1050: footprint Package_DIP:DIP-8_W7.62mm_LongPads -> LIbCapteurPCB:LTC1050
- moved Flex1 39.1 mm to (120.0, 92.0)
- moved MCP1 23.9 mm to (147.0, 85.5), turned to 0 degrees
- moved C2 18.9 mm to (138.7, 69.5)
- moved C3 15.6 mm to (133.7, 65.5)
- moved R5 15.2 mm to (138.3, 66.0)
- moved LTC1050 15.2 mm to (125.0, 66.5)
- moved C4 11.2 mm to (124.3, 58.0)
- moved R3 9.00 mm to (133.7, 69.0)
- moved OLED1 8.67 mm to (161.0, 82.7)
- moved R4 8.32 mm to (117.5, 75.0)
- moved C1 8.10 mm to (121.0, 77.0), turned to 90 degrees
- moved R2 7.09 mm to (127.7, 77.0), turned to 90 degrees
- moved R1 6.50 mm to (124.0, 77.0), turned to 90 degrees
- moved BT1 5.75 mm to (140.7, 58.0), turned to 180 degrees
Connections:
- net /LED_D11 renamed /*11
- net /LED_D12 renamed /12
- BT1 pad 1: unconnected-(BT1-5V-Pad1) -> +5V
- BT1 pad 2: unconnected-(BT1-GND-Pad2) -> GND
- BT1 pad 3: unconnected-(BT1-Tx-Pad3) -> B-3: Tx
- BT1 pad 4: unconnected-(BT1-RX-Pad4) -> B-4: Rx
- Flex1 pad 1: unconnected-(Flex1-Pad1) -> +5V
- Flex1 pad 2: unconnected-(Flex1-Pad2) -> F-2
- J2 pad 10: /8 -> B-3: Tx
- J2 pad 8: /LED_D10 -> M-1: CS
- J2 pad 9: /LED_D9 -> B-4: Rx
- J3 pad 2: /A1 -> F-2
- J3 pad 5: /SDA/A4 -> O-4: SDA
- J3 pad 6: /SCL/A5 -> O-3: SCL
- J4 pad 3: /*5 -> R-3: SWITCH
- J4 pad 4: /4 -> R-2: DATA
- J4 pad 6: /2 -> R-1: CLK
- MCP1 pad 1: unconnected-(MCP1-CS-Pad1) -> M-1: CS
- MCP1 pad 2: unconnected-(MCP1-SCK-Pad2) -> M-2: SCK
- MCP1 pad 3: unconnected-(MCP1-SI-Pad3) -> M-3: SI
- MCP1 pad 4: unconnected-(MCP1-VSS-Pad4) -> GND
- MCP1 pad 5: unconnected-(MCP1-A-Pad5) -> M-5: A
- MCP1 pad 6: unconnected-(MCP1-W-Pad6) -> M-6: W
- MCP1 pad 7: unconnected-(MCP1-B-Pad7) -> M-7: B
- MCP1 pad 8: unconnected-(MCP1-VCC-Pad8) -> +5V
- OLED1 pad 1: unconnected-(OLED1-GND-Pad1) -> GND
- OLED1 pad 2: unconnected-(OLED1-+5V-Pad2) -> +5V
- OLED1 pad 3: unconnected-(OLED1-SCL-Pad3) -> O-3: SCL
- OLED1 pad 4: unconnected-(OLED1-SDA-Pad4) -> O-4: SDA
Routing:
- removed copper zone on B.Cu, net GND
Other:
- board text removed: "delcampo@insa-toulouse.fr"
