File: KiCad/ProjetCpatKiCad/ProjetCpatKiCad/ProjetCpatKiCad.kicad_pcb (KiCad board)
At the start: 2 copper layers, 68.6 x 53.3 mm, 24 parts, among them J1 Power, J2 Digital/PWM, J3 Analog, J4 Digital/PWM

Commit message: tiqui
Parts:
- C1, C2, C3: footprint Capacitor_SMD:C_0201_0603Metric -> Capacitor_THT:C_Axial_L3.8mm_D2.6mm_P7.50mm_Horizontal
- C4: footprint Capacitor_SMD:C_0201_0603Metric -> Capacitor_THT:C_Rect_L4.6mm_W5.5mm_P2.50mm_MKS02_FKP02
- R1, R2, R3, R4, R5: footprint Resistor_SMD:R_0201_0603Metric -> Resistor_THT:R_Axial_DIN0204_L3.6mm_D1.6mm_P1.90mm_Vertical
- moved Flex1 25.8 mm to (145.8, 91.0)
- moved MCP1 16.5 mm to (147.0, 69.0), turned to 180 degrees
- moved C2 16.2 mm to (141.2, 85.5), turned to 180 degrees
- moved R3 14.9 mm to (123.5, 58.1), turned to -90 degrees
- moved R5 13.5 mm to (139.0, 79.5), turned to -90 degrees
- moved C4 12.7 mm to (119.0, 69.5), turned to 180 degrees
- moved C3 11.7 mm to (128.0, 55.2), turned to -90 degrees
- moved C1 8.53 mm to (120.2, 85.5), turned to 0 degrees
- moved R2 5.92 mm to (133.0, 79.6), turned to -90 degrees
- moved R1 4.77 mm to (128.0, 79.6), turned to -90 degrees
- moved R4 4.30 mm to (120.0, 78.5)
- moved BT1 4.03 mm to (144.2, 56.0)
- moved LTC1050 4.03 mm to (127.0, 70.0), turned to 90 degrees
- moved CAP1 3.64 mm to (112.5, 70.0)
- moved ROT1 3.50 mm to (158.5, 58.0)
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Connections:
- J2 pad 5: /13 -> M-2: SCK
- J2 pad 7: /*11 -> M-3: SI
- J3 pad 1: ADC -> F-2
- J3 pad 2: F-2 -> ADC
- MCP1 pad 4: GND -> unconnected-(MCP1-VSS-Pad4)
- MCP1 pad 8: +5V -> unconnected-(MCP1-VCC-Pad8)
Routing:
- net +5V: track 0.00 -> 149.4 mm, vias 0 -> 6
- net GND: track 0.00 -> 103.8 mm
- net Net-(LTC1050-OUT): track 0.00 -> 60.2 mm
- net M-2: SCK: track 0.00 -> 32.2 mm
- net Net-(LTC1050-+IN): track 0.00 -> 31.9 mm
- net M-1: CS: track 0.00 -> 26.0 mm
- net ADC: track 0.00 -> 25.0 mm
- net Net-(LTC1050--IN): track 0.00 -> 24.9 mm
- net M-3: SI: track 0.00 -> 22.8 mm
- net O-3: SCL: track 0.00 -> 15.3 mm
- net R-2: DATA: track 0.00 -> 12.5 mm
- net R-3: SWITCH: track 0.00 -> 12.0 mm
- net O-4: SDA: track 0.00 -> 11.0 mm
- net R-1: CLK: track 0.00 -> 10.9 mm
- net Net-(CAP1-GND): track 0.00 -> 9.90 mm
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- added copper zone on B.Cu, net GND

Commit message: Kicad routage
Parts:
- removed R2: 1k, Resistor_THT:R_Axial_DIN0204_L3.6mm_D1.6mm_P1.90mm_Vertical
- Flex1: footprint LIbCapteurPCB:F_SENSE -> ChuloPCB:Flexeo
- moved Flex1 6.77 mm to (139.0, 91.5), turned to -90 degrees
- moved C3 2.00 mm to (126.0, 55.2)
- moved R3 2.00 mm to (121.5, 58.1)
Connections:
- C1 pad 1: Net-(LTC1050-+IN) -> M-7: B
- LTC1050 pad 3: Net-(LTC1050-+IN) -> M-7: B
- MCP1 pad 6: M-6: W -> GND
- R1 pad 1: Net-(LTC1050-+IN) -> M-7: B
- R4 pad 2: Net-(LTC1050-+IN) -> M-7: B
Routing:
- net M-7: B: track 0.00 -> 50.6 mm
- net Net-(LTC1050-+IN): track 31.9 -> 0.00 mm
- net +5V: track 149.4 -> 177.3 mm, vias 6 -> 0
- net Net-(LTC1050-OUT): track 60.2 -> 87.9 mm
- net GND: track 103.8 -> 100.3 mm
- net F-2: track 9.21 -> 10.3 mm
- net Net-(LTC1050--IN): track 24.9 -> 24.0 mm

Commit message: VIA GND
Routing:
- net GND: track 100.3 -> 134.6 mm, vias 0 -> 2
Changed lines of the file:
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@@
+	)
+	(segment
+		(start 157 73.5)
+		(end 161 73.5)
+		(width 0.8)
+		(layer "F.Cu")
+		(net 1)
+	)
+	(segment
+		(start 138 75.5)
+		(end 139 76.5)
+		(width 0.8)
+		(layer "F.Cu")
+		(net 1)
+	)
+	(segment
+		(start 139 76.5)
+		(end 154 76.5)
+		(width 0.8)
+		(layer "F.Cu")
+		(net 1)
+	)
+	(segment
+		(start 138 71.56)
+		(end 138 75.5)
+		(width 0.8)
+		(layer "F.Cu")
+		(net 1)
+	)
+	(segment
+		(start 154 76.5)
+		(end 157 73.5)
+		(width 0.8)
+		(layer "F.Cu")
+		(net 1)
+	)
+	(segment
+		(start 137.72 71.28)
+		(end 138 71.56)
+		(width 0.8)
+		(layer "F.Cu")
+		(net 1)
+	)
+	(via
+		(at 161 73.5)
+		(size 2.2)
+		(drill 0.8)
+		(layers "F.Cu" "B.Cu")
+		(net 1)
+	)
+	(via
+		(at 137.72 71.28)
+		(size 2.2)
+		(drill 0.8)
+		(layers "F.Cu" "B.Cu")
+		(net 1)
+	)
+	(segment
+		(start 145.73 74.09)
+		(end 144.79 75.03)
+		(width 0.6)
+		(layer "B.Cu")
+		(net 1)
 	)
 	(segment
@@
 	)
 	(segment
-		(start 145.73 74.09)
-		(end 144.79 75.03)
+		(start 140.64 97.46)
+		(end 140.64 92.87)
+		(width 0.6)
+		(layer "B.Cu")
+		(net 1)
+	)
+	(segment
+		(start 145.73 72.76)
+		(end 145.73 74.09)
 		(width 0.6)
 		(layer "B.Cu")
@@
 	)
 	(segment
-		(start 140.64 97.46)
-		(end 140.64 92.87)
-		(width 0.6)
-		(layer "B.Cu")
-		(net 1)
-	)
-	(segment
-		(start 145.73 72.76)
-		(end 145.73 74.09)
-		(width 0.6)
-		(layer "B.Cu")
-		(net 1)
-	)
-	(segment
 		(start 127.75 87.75)
 		(end 127.75 85.5)
@@
 	)
 	(segment
+		(start 128 81.495)
+		(end 128 85.25)
+		(width 0.6)
+		(layer "B.Cu")
+		(net 1)
+	)
+	(segment
 		(start 144.79 75.03)
 		(end 141.47 75.03)
@@
 	)
 	(segment
-		(start 128 81.495)
-		(end 128 85.25)
-		(width 0.6)
-		(layer "B.Cu")
-		(net 1)
-	)
-	(segment
 		(start 116.5 69.5)
 		(end 111.5 69.5)
@@
 		(layer "B.Cu")
 		(net 1)
+	)
+	(segment
+		(start 161 73.5)
+		(end 161 78.88)
+		(width 0.8)
+		(layer "B.Cu")
+		(net 1)

Commit message: Kicad modelos 3d
Parts:
- moved BT1 1.54 mm to (142.7, 56.0)
Routing:
- net ADC: track 25.0 -> 34.0 mm
- net Net-(LTC1050-OUT): track 87.9 -> 91.1 mm
- net M-1: CS: track 26.0 -> 27.8 mm
- net M-3: SI: track 22.8 -> 24.6 mm
- net GND: track 134.6 -> 136.1 mm
- net +5V: track 177.3 -> 178.4 mm

Commit message: Kicad con servo
Parts:
- added SV1: ~, ChuloPCB:SIP-3, F.Cu at (146.5, 53.5)
- moved BT1 3.20 mm to (144.7, 58.5)
- turned OLED1 to 90 degrees
Connections:
- J4 pad 2: /*6 -> Dig
Routing:
- net GND: track 136.1 -> 105.2 mm, vias 2 -> 0
- net O-4: SDA: track 11.0 -> 26.0 mm
- net +5V: track 178.4 -> 189.5 mm
- net O-3: SCL: track 15.3 -> 23.4 mm
- net Dig: track 0.00 -> 4.61 mm
- net B-3: Tx: track 6.90 -> 10.0 mm
- net B-4: Rx: track 6.90 -> 10.0 mm
- net M-1: CS: track 27.8 -> 29.0 mm
- net Net-(LTC1050-OUT): track 91.1 -> 89.9 mm

Commit message: kikadfinal
Dale visto bueno
Parts:
- moved SV1 48.7 mm to (103.5, 76.5), turned to -90 degrees
- moved BT1 2.66 mm to (142.6, 56.8)
Routing:
- net Dig: track 4.61 -> 63.3 mm, vias 0 -> 2
- net GND: track 105.2 -> 117.4 mm, vias 0 -> 2
- net B-3: Tx: track 10.0 -> 7.74 mm
- net B-4: Rx: track 10.0 -> 7.74 mm
- net M-1: CS: track 29.0 -> 27.7 mm
- net M-7: B: track 50.6 -> 51.7 mm
