File: KiCad/ProjetCpatKiCad_DELCAMPO_VALENCIA/ProjetCpatKiCad/ProjetCpatKiCad.kicad_pcb (KiCad board)
At the start: 2 copper layers, 68.6 x 53.3 mm, 24 parts, among them J1 Power, J2 Digital/PWM, J3 Analog, J4 Digital/PWM

Commit message: Changes PINS R et C
Other:
- board text added: "DEL CAMPO VALENCIA"
Changed lines of the file:
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@@
 			)
 		)
-		(pad "1" thru_hole circle
+		(pad "1" thru_hole oval
 			(at 0 0 270)
-			(size 1.4 1.4)
+			(size 1.5 2.54)
 			(drill 0.7)
 			(layers "*.Cu" "*.Mask")
@@
 		(pad "2" thru_hole oval
 			(at 1.9 0 270)
-			(size 1.4 1.4)
+			(size 1.5 2.54)
 			(drill 0.7)
 			(layers "*.Cu" "*.Mask")
@@
 			)
 		)
-		(pad "1" thru_hole circle
+		(pad "1" thru_hole oval
 			(at 0 0 180)
-			(size 1.6 1.6)
+			(size 2 2.54)
 			(drill 0.8)
 			(layers "*.Cu" "*.Mask")
@@
 		(pad "2" thru_hole oval
 			(at 7.5 0 180)
-			(size 1.6 1.6)
+			(size 2 2.54)
 			(drill 0.8)
 			(layers "*.Cu" "*.Mask")
@@
 			)
 		)
-		(pad "1" thru_hole circle
+		(pad "1" thru_hole oval
 			(at 0 0 270)
-			(size 1.6 1.6)
+			(size 2 2.54)
 			(drill 0.8)
 			(layers "*.Cu" "*.Mask")
@@
 		(pad "2" thru_hole oval
 			(at 7.5 0 270)
-			(size 1.6 1.6)
+			(size 2 2.54)
 			(drill 0.8)
 			(layers "*.Cu" "*.Mask")
@@
 			)
 		)
-		(pad "1" thru_hole circle
+		(pad "1" thru_hole oval
 			(at 0 0 270)
-			(size 1.4 1.4)
+			(size 1.4 2.54)
 			(drill 0.7)
 			(layers "*.Cu" "*.Mask")
@@
 		(pad "2" thru_hole oval
 			(at 1.9 0 270)
-			(size 1.4 1.4)
+			(size 1.4 2.54)
 			(drill 0.7)
 			(layers "*.Cu" "*.Mask")
@@
 			)
 		)
-		(pad "1" thru_hole circle
+		(pad "1" thru_hole oval
 			(at 0 0)
-			(size 1.6 1.6)
+			(size 2 2.54)
 			(drill 0.8)
 			(layers "*.Cu" "*.Mask")
@@
 		(pad "2" thru_hole oval
 			(at 7.5 0)
-			(size 1.6 1.6)
+			(size 2 2.54)
 			(drill 0.8)
 			(layers "*.Cu" "*.Mask")
@@
 			)
 		)
-		(pad "1" thru_hole circle
+		(pad "1" thru_hole oval
 			(at 0 0 270)
-			(size 1.4 1.4)
+			(size 1.4 2.54)
 			(drill 0.7)
 			(layers "*.Cu" "*.Mask")
@@
 		(pad "2" thru_hole oval
 			(at 1.9 0 270)
-			(size 1.4 1.4)
+			(size 1.4 2.54)
 			(drill 0.7)
 			(layers "*.Cu" "*.Mask")
@@
 			)
 		)
-		(pad "1" thru_hole circle
+		(pad "1" thru_hole oval
 			(at 0 0 180)
-			(size 1.4 1.4)
+			(size 1.9 2.54)
 			(drill 0.7)
 			(layers "*.Cu" "*.Mask")
@@
 			(pintype "passive")
 		)
-		(pad "2" thru_hole circle
+		(pad "2" thru_hole oval
 			(at 2.5 0 180)
-			(size 1.4 1.4)
+			(size 1.9 2.54)
 			(drill 0.7)
-			(layers "*.Cu" "*.Mask")
+			(layers "*.Cu" "*.Mask" "Eco2.User")
 			(remove_unused_layers no)
 			(net 1 "GND")
@@
 			)
 		)
-		(pad "1" thru_hole circle
+		(pad "1" thru_hole oval
 			(at 0 0)
-			(size 1.4 1.4)
+			(size 1.4 2.54)
 			(drill 0.7)
 			(layers "*.Cu" "*.Mask")
@@
 		(pad "2" thru_hole oval
 			(at 1.9 0)
-			(size 1.4 1.4)
+			(size 1.4 2.54)
 			(drill 0.7)
 			(layers "*.Cu" "*.Mask")
@@
 		(layer "Edge.Cuts")
 	)
+	(gr_text "DEL CAMPO\nVALENCIA"
+		(at 101.893084 60.9 -90)
+		(layer "B.Cu")
+		(effects
+			(font
+				(size 1.5 1.5)
+				(thickness 0.3)
+				(bold yes)
+			)
+			(justify left bottom mirror)
+		)
+	)
 	(gr_text "ICSP"
